Commit message: initial

File: src/arm_control/config/robot_arm.urdf (robot description, URDF)
Before this commit: robot arm, 7 links, 8 joints
Links:
- added link hand_left_link, mass 1; collision box size=0.1 0.05 0.1; visual box size=0.1 0.05 0.1
- added link hand_right_link, mass 1; collision box size=0.1 0.05 0.1; visual box size=0.1 0.05 0.1
Joints:
- joint hand_left_joint: limit lower=0 upper=0.05 effort=3000 velocity=0.03 -> lower=0 upper=0.05 effort=3000.0 velocity=0.03; origin xyz=0 0.075 0.05 rpy=0 0 0 -> xyz=0.0 0.075 0.05 rpy=0.0 0.0 0.0
- joint hand_right_joint: limit lower=0 upper=0.05 effort=3000 velocity=0.03 -> lower=0 upper=0.05 effort=3000.0 velocity=0.03; origin xyz=0 -0.075 0.05 rpy=0 0 0 -> xyz=0.0 -0.075 0.05 rpy=0.0 0.0 0.0
- joint joint1: limit lower=-3.14 upper=3.14 effort=100 velocity=1 -> lower=-3.14 upper=3.14 effort=100.0 velocity=1; origin xyz=0 0 0.1 rpy=0 0 0 -> xyz=0.0 0.0 0.1 rpy=0.0 0.0 0.0
- joint joint2: limit lower=-3.14 upper=3.14 effort=100 velocity=1 -> lower=-3.14 upper=3.14 effort=100.0 velocity=1; origin xyz=0 0 0.1 rpy=0 0 0 -> xyz=0.0 0.0 0.1 rpy=0.0 0.0 0.0
- joint joint3: limit lower=-3.14 upper=3.14 effort=100 velocity=1 -> lower=-3.14 upper=3.14 effort=100.0 velocity=1; origin xyz=0 0 0.3 rpy=0 0 0 -> xyz=0.0 0.0 0.3 rpy=0.0 0.0 0.0
- joint joint4: limit lower=-3.14 upper=3.14 effort=100 velocity=1 -> lower=-3.14 upper=3.14 effort=100.0 velocity=1; origin xyz=0 0 0.3 rpy=0 0 0 -> xyz=0.0 0.0 0.3 rpy=0.0 0.0 0.0
- joint joint5: limit lower=-3.14 upper=3.14 effort=100 velocity=1 -> lower=-3.14 upper=3.14 effort=100.0 velocity=1; origin xyz=0 0 0.3 rpy=0 0 0 -> xyz=0.0 0.0 0.3 rpy=0.0 0.0 0.0
- joint joint6: limit lower=-3.14 upper=3.14 effort=100 velocity=1 -> lower=-3.14 upper=3.14 effort=100.0 velocity=1; origin xyz=0 0 0.3 rpy=0 0 0 -> xyz=0.0 0.0 0.3 rpy=0.0 0.0 0.0
