Commit message: 添加dummy_control文件

File: src/dummy_control/config/dummy_ros2_control.xacro (robot description, xacro)
@@ -26,60 +26,103 @@
       </xacro:unless>
     </hardware>
-    <!-- joint1 -->
-    <joint name="joint1">
-      <command_interface name="position"/>
+  <!-- Gazebo material tags -->
+  <gazebo reference="Base_Link">
+    <material>Gazebo/Grey</material>
+    <gravity>true</gravity>
+    <selfCollide>false</selfCollide>
+  </gazebo>
+  <gazebo reference="Link1">
+    <material>Gazebo/Gray</material>
+    <selfCollide>false</selfCollide>
+  </gazebo>
+  <gazebo reference="Link2">
+    <material>Gazebo/Grey</material>
+    <selfCollide>false</selfCollide>
+  </gazebo>
+  <gazebo reference="Link3">
+    <material>Gazebo/Grey</material>
+  </gazebo>
+  <gazebo reference="Link4">
+    <material>Gazebo/Grey</material>
+  </gazebo>
+  <gazebo reference="Link5">
+    <material>Gazebo/Grey</material>
+  </gazebo>
+  <gazebo reference="Link6">
+    <material>Gazebo/DarkGrey</material>
+  </gazebo>
+  <!-- ros2_control configuration for Gazebo -->
+  <ros2_control name="GazeboSystem" type="system">
+    <hardware>
+      <plugin>gazebo_ros2_control/GazeboSystem</plugin>
+    </hardware>
+    <joint name="Joint1">
+      <command_interface name="position">
+        <param name="min">-1</param>
+        <param name="max">1</param>
+      </command_interface>
       <state_interface name="position">
-        <param name="initial_value">0</param>
+        <param name="initial_value">0.0</param>
       </state_interface>
       <state_interface name="velocity"/>
     </joint>
-    <!-- joint2 -->
-    <joint name="joint2">
-      <command_interface name="position"/>
+    <joint name="Joint2">
+      <command_interface name="position">
+        <param name="min">-1</param>
+        <param name="max">1</param>
+      </command_interface>
       <state_interface name="position">
-        <param name="initial_value">0</param>
+        <param name="initial_value">0.0</param>
       </state_interface>
       <state_interface name="velocity"/>
     </joint>
-    <!-- joint3 -->
-    <joint name="joint3">
-      <command_interface name="position"/>
+    <joint name="Joint3">
+      <command_interface name="position">
+        <param name="min">-1</param>
+        <param name="max">1</param>
+      </command_interface>
       <state_interface name="position">
-        <param name="initial_value">0</param>
+        <param name="initial_value">0.0</param>
       </state_interface>
       <state_interface name="velocity"/>
     </joint>
-    <!-- joint4 -->
-    <joint name="joint4">
-      <command_interface name="position"/>
+    <joint name="Joint4">
+      <command_interface name="position">
+        <param name="min">-1</param>
+        <param name="max">1</param>
+      </command_interface>
       <state_interface name="position">
-        <param name="initial_value">0</param>
+        <param name="initial_value">0.0</param>
       </state_interface>
       <state_interface name="velocity"/>
     </joint>
-    <!-- joint5 -->
-    <joint name="joint5">
-      <command_interface name="position"/>
+    <joint name="Joint5">
+      <command_interface name="position">
+        <param name="min">-1</param>
+        <param name="max">1</param>
+      </command_interface>
       <state_interface name="position">
-        <param name="initial_value">0</param>
+        <param name="initial_value">0.0</param>
       </state_interface>
       <state_interface name="velocity"/>
     </joint>
-    <!-- joint6 -->
-    <joint name="joint6">
-      <command_interface name="position"/>
+    <joint name="Joint6">
+      <command_interface name="position">
+        <param name="min">-1</param>
+        <param name="max">1</param>
+      </command_interface>
       <state_interface name="position">
-        <param name="initial_value">0</param>
-      </state_interface>
-      <state_interface name="velocity"/>
-    </joint>
-    <!-- gripper -->
-    <joint name="hand_right_joint">
-      <command_interface name="position"/>
-      <state_interface name="position">
-        <param name="initial_value">0</param>
+        <param name="initial_value">0.0</param>
       </state_interface>
       <state_interface name="velocity"/>
     </joint>
   </ros2_control>
+  <!-- Gazebo ros2_control plugin -->
+  <gazebo>
+    <plugin filename="libgazebo_ros2_control.so" name="gazebo_ros2_control">
+      <parameters>$(find mydummy)/config/ros2_controllers.yaml</parameters>
+      <robot_param_node>robot_state_publisher</robot_param_node>
+    </plugin>
+  </gazebo>
+  </ros2_control>
 </robot>

File: src/dummy_control/config/mydummy.urdf (robot description, URDF)
Before this commit: robot mydummy_description, 8 links, 7 joints
Links:
- removed link world
Joints:
- removed joint fixed

Commit message: 添加dummy_control文件

File: src/dummy_control/config/dummy_ros2_control.xacro (robot description, xacro)
@@ -1,29 +1,6 @@
 <?xml version="1.0" encoding="UTF-8"?>
-<robot xmlns:xacro="http://www.ros.org/wiki/xacro" name="arm">
+<robot xmlns:xacro="http://www.ros.org/wiki/xacro" name="mydummy">
   <xacro:arg name="use_gazebo" default="false"/>
-  <xacro:include filename="robot_arm.urdf"/>
-  <!-- 是否添加 gz_ros2_control-system -->
-  <xacro:if value="$(arg use_gazebo)">
-    <gazebo>
-      <!-- 添加 world-joint 使机械臂固定在 Gazebo 仿真场景中 -->
-      <joint name="world_joint" type="fixed">
-        <parent>world</parent>
-        <child>base_link</child>
-      </joint>
-      <plugin filename="gz_ros2_control-system"
-              name="gz_ros2_control::GazeboSimROS2ControlPlugin">
-        <parameters>$(find arm_control)/config/arm_controllers.yaml</parameters>
-      </plugin>
-    </gazebo>
-  </xacro:if>
-  <ros2_control name="MyRobotSystem" type="system">
-    <hardware>
-      <xacro:if value="$(arg use_gazebo)">
-        <plugin>gz_ros2_control/GazeboSimSystem</plugin>
-      </xacro:if>
-      <xacro:unless value="$(arg use_gazebo)">
-        <plugin>mock_components/GenericSystem</plugin>
-      </xacro:unless>
-    </hardware>
+  <xacro:include filename="mydummy.urdf"/>
   <!-- Gazebo material tags -->
   <gazebo reference="Base_Link">
@@ -52,77 +29,75 @@
     <material>Gazebo/DarkGrey</material>
   </gazebo>
-  <!-- ros2_control configuration for Gazebo -->
-  <ros2_control name="GazeboSystem" type="system">
+  <!-- 是否添加 gz_ros2_control-system -->
+  <xacro:if value="$(arg use_gazebo)">
+    <gazebo>
+      <!-- 添加 world-joint 使机械臂固定在 Gazebo 仿真场景中 -->
+      <joint name="world_joint" type="fixed">
+        <parent>world</parent>
+        <child>Base_Link</child>
+      </joint>
+      <plugin filename="gz_ros2_control-system"
+              name="gz_ros2_control::GazeboSimROS2ControlPlugin">
+        <parameters>$(find dummy_control)/config/dummy_controllers.yaml</parameters>
+      </plugin>
+    </gazebo>
+  </xacro:if>
+  <ros2_control name="MyDummySystem" type="system">
     <hardware>
-      <plugin>gazebo_ros2_control/GazeboSystem</plugin>
+      <xacro:if value="$(arg use_gazebo)">
+        <plugin>gz_ros2_control/GazeboSimSystem</plugin>
+      </xacro:if>
+      <xacro:unless value="$(arg use_gazebo)">
+        <plugin>mock_components/GenericSystem</plugin>
+      </xacro:unless>
     </hardware>
+    <!-- Joint1 -->
     <joint name="Joint1">
-      <command_interface name="position">
-        <param name="min">-1</param>
-        <param name="max">1</param>
-      </command_interface>
+      <command_interface name="position"/>
       <state_interface name="position">
-        <param name="initial_value">0.0</param>
+        <param name="initial_value">0</param>
       </state_interface>
       <state_interface name="velocity"/>
     </joint>
+    <!-- Joint2 -->
     <joint name="Joint2">
-      <command_interface name="position">
-        <param name="min">-1</param>
-        <param name="max">1</param>
-      </command_interface>
+      <command_interface name="position"/>
       <state_interface name="position">
-        <param name="initial_value">0.0</param>
+        <param name="initial_value">0</param>
       </state_interface>
       <state_interface name="velocity"/>
     </joint>
+    <!-- Joint3 -->
     <joint name="Joint3">
-      <command_interface name="position">
-        <param name="min">-1</param>
-        <param name="max">1</param>
-      </command_interface>
+      <command_interface name="position"/>
       <state_interface name="position">
-        <param name="initial_value">0.0</param>
+        <param name="initial_value">0</param>
       </state_interface>
       <state_interface name="velocity"/>
     </joint>
+    <!-- Joint4 -->
     <joint name="Joint4">
-      <command_interface name="position">
-        <param name="min">-1</param>
-        <param name="max">1</param>
-      </command_interface>
+      <command_interface name="position"/>
       <state_interface name="position">
-        <param name="initial_value">0.0</param>
+        <param name="initial_value">0</param>
       </state_interface>
       <state_interface name="velocity"/>
     </joint>
+    <!-- Joint5 -->
     <joint name="Joint5">
-      <command_interface name="position">
-        <param name="min">-1</param>
-        <param name="max">1</param>
-      </command_interface>
+      <command_interface name="position"/>
       <state_interface name="position">
-        <param name="initial_value">0.0</param>
+        <param name="initial_value">0</param>
       </state_interface>
       <state_interface name="velocity"/>
     </joint>
+    <!-- Joint6 -->
     <joint name="Joint6">
-      <command_interface name="position">
-        <param name="min">-1</param>
-        <param name="max">1</param>
-      </command_interface>
+      <command_interface name="position"/>
       <state_interface name="position">
-        <param name="initial_value">0.0</param>
+        <param name="initial_value">0</param>
       </state_interface>
       <state_interface name="velocity"/>
     </joint>
   </ros2_control>
-  <!-- Gazebo ros2_control plugin -->
-  <gazebo>
-    <plugin filename="libgazebo_ros2_control.so" name="gazebo_ros2_control">
-      <parameters>$(find mydummy)/config/ros2_controllers.yaml</parameters>
-      <robot_param_node>robot_state_publisher</robot_param_node>
-    </plugin>
-  </gazebo>
-  </ros2_control>
 </robot>

File: src/dummy_control/config/mydummy.urdf (robot description, URDF)
Before this commit: robot mydummy_description, 7 links, 6 joints
Links:
- link Base_Link: geometry collision mesh filename=file:///home/jiehuang/arm_control_ws/src/dummy_control/mesh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; visual mesh filename=file:///home/jiehuang/arm_control_ws/src/dummy_control/mesh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
- link Link1: geometry collision mesh filename=file:///home/jiehuang/arm_control_ws/src/dummy_control/mesh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; visual mesh filename=file:///home/jiehuang/arm_control_ws/src/dummy_control/mesh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
- link Link2: geometry collision mesh filename=file:///home/jiehuang/arm_control_ws/src/dummy_control/mesh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; visual mesh filename=file:///home/jiehuang/arm_control_ws/src/dummy_control/mesh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
- link Link3: geometry collision mesh filename=file:///home/jiehuang/arm_control_ws/src/dummy_control/mesh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; visual mesh filename=file:///home/jiehuang/arm_control_ws/src/dummy_control/mesh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
- link Link4: geometry collision mesh filename=file:///home/jiehuang/arm_control_ws/src/dummy_control/mesh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; visual mesh filename=file:///home/jiehuang/arm_control_ws/src/dummy_control/mesh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
- link Link5: geometry collision mesh filename=file:///home/jiehuang/arm_control_ws/src/dummy_control/mesh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; visual mesh filename=file:///home/jiehuang/arm_control_ws/src/dummy_control/mesh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
- link Link6: geometry collision mesh filename=file:///home/jiehuang/arm_control_ws/src/dummy_control/mesh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; visual mesh filename=file:///home/jiehuang/arm_control_ws/src/dummy_control/mesh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
